File: light_blade/light_blade.kicad_pcb (KiCad board)
At the start: 2 copper layers, 356 x 65 mm, 68 parts, among them J1 IN, J2 OUT, M3 MountingHole_3.2mm_M3, U1 WS2811, U10 WS2811, U2 WS2811, U3 WS2811, U4 WS2811, U5 WS2811, U6 WS2811, U7 WS2811, U8 WS2811, U9 WS2811

Commit message: Rev 3: mounting-hole keepouts, decoupling fixes, D17/D18 in schematic
- Add copper keepouts on both layers around all mounting holes
  (7 mm for M3, 11 mm for M5) so metal screws can't bridge +5V/GND
- Move C6 and C7 next to the VDD pin of U6/U7 (was ~10 mm away);
  R7 moved back to its standard position to make room
- Add D17/D18 to the schematic on U4_G/U4_B and link the PCB
  footprints, removing the U4 schematic/PCB net conflicts
- Regenerate fab_gerber and a new PCBWay export (2026-10-18) with
  BOM Rev 3 and positions file
- Update plan doc for U4 driving D10/D17/D18

Co-Authored-By: Claude Opus 5.5 <noreply@anthropic.com>
Parts:
- moved C6 10.8 mm to (196.5, 95.0), turned to 0 degrees
- moved C7 7.21 mm to (228.4, 90.6), turned to 180 degrees
- moved R7 1.60 mm to (228.0, 88.4)
Routing:
- net Net-(U7-VDD): track 14.8 -> 17.0 mm
- net GND: track 36.9 -> 34.8 mm
- net Net-(U6-VDD): track 12.7 -> 13.7 mm
- net /DATA6: track 37.0 -> 37.7 mm
- net Net-(U7-DIN): track 3.27 -> 2.61 mm
