File: light_blade/light_blade.kicad_sch (KiCad schematic)
At the start: 60 parts, among them J1 IN, J2 OUT, U1 WS2811, U10 WS2811, U2 WS2811, U3 WS2811, U4 WS2811, U5 WS2811, U6 WS2811, U7 WS2811, U8 WS2811, U9 WS2811

Commit message: Rev 3: mounting-hole keepouts, decoupling fixes, D17/D18 in schematic
- Add copper keepouts on both layers around all mounting holes
  (7 mm for M3, 11 mm for M5) so metal screws can't bridge +5V/GND
- Move C6 and C7 next to the VDD pin of U6/U7 (was ~10 mm away);
  R7 moved back to its standard position to make room
- Add D17/D18 to the schematic on U4_G/U4_B and link the PCB
  footprints, removing the U4 schematic/PCB net conflicts
- Regenerate fab_gerber and a new PCBWay export (2026-10-18) with
  BOM Rev 3 and positions file
- Update plan doc for U4 driving D10/D17/D18

Co-Authored-By: Claude Opus 5.5 <noreply@anthropic.com>
Parts:
- added D17, D18: LED 0805 white, LED_SMD:LED_0805_2012Metric, symbol Device:LED
Connections:
- net +5V: now also D17.2 (A), D18.2 (A)
- net U4_G: now reaches U4.2 (OUTG)
- net U4_G: now also D17.1 (K)
- net U4_B: now reaches U4.3 (OUTB)
- net U4_B: now also D18.1 (K)
- no-connect marks 12 -> 10
